File: SpiderBotPCB/SpiderBotPCB.kicad_sch (KiCad schematic)
At the start: 12 parts, among them U1 STM32L412KBT6, U2 L7986A

Commit message: add stuff
Parts:
- added D2: LED_PWR_STATUS, symbol Device:LED
- added M1, M10, M11, M12, M2, M3, M4, M5, M6, M7, M8, M9: Motor_Servo, symbol Motor:Motor_Servo
- added R5: 1k5, symbol Device:R
- added U3: HT7533-1, HT7533-1:SOT89, symbol HT7533:HT7533-1
Connections:
- net +3.3V: no longer C2.2, L1.2, R1.1
- net GND: now also D2.1 (K), M1.3 (-), M10.3 (-), M11.3 (-), M12.3 (-), M2.3 (-), M3.3 (-), M4.3 (-), M5.3 (-), M6.3 (-), M7.3 (-), M8.3 (-), M9.3 (-)
- new net: U3.2 (VI), U3.2@1 (VI)
- new net: D2.2 (A), R5.2
- new net +4.8V: C2.2, L1.2, M1.2 (+), M10.2 (+), M11.2 (+), M12.2 (+), M2.2 (+), M3.2 (+), M4.2 (+), M5.2 (+), M6.2 (+), M7.2 (+), M8.2 (+), M9.2 (+), R1.1, R5.1
Other:
- note added: "4.8V step down from battery"
- moved on the sheet: U1

Commit message: finish power circuits on the PCB
Parts:
- removed C2: 100u, symbol Device:C
- added C10, C11, C5, C7, C8, C9: 470u, symbol Device:C_Polarized
- added C12: 1u, symbol Device:C
- added C13: 47u, symbol Device:C_Polarized
- added C14: 0.01u, symbol Device:C
- added C15: 0.1p, symbol Device:C
- added C16: 330p, symbol Device:C
- added C17, C18, C2: 100u, symbol Device:C_Polarized
- added C6: 10u, symbol Device:C
- added D3: D_Schottky, symbol Device:D_Schottky
- added J1: Jack-DC, symbol Connector:Jack-DC
- added L2: 33u, symbol Device:L
- added U4: ST763A, Package_SO:SO-8_3.9x4.9mm_P1.27mm, symbol ST763A:ST763A
- renumbered U3 to U3-stabilizer
Connections:
- net +12.6V: now also J1.1
- net +3.3V: now also U3-stabilizer.3 (VO), C18.1
- net +4.8V: now also C10.1, C11.1, C12.2, C13.1, C2.1, C5.1, C6.2, C7.1, C8.1, C9.1, U4.1 (SHDN), U4.8 (VCC)
- net GND: now also U3-stabilizer.1, C10.2, C11.2, C12.1, C13.2, C14.1, C15.1, C17.2, C18.2, C2.2, C5.2, C6.1, C7.2, C8.2, C9.2, D3.2 (A), J1.2, U4.6 (GND)
- net at U3-stabilizer.2 (VI), U3-stabilizer.2@1 (VI): now also C16.2, C17.1, L2.2, U4.5 (OUT)
- new net: D3.1 (K), L2.1, U4.7 (LX)
- new net: C16.1, U4.4 (CC)
- new net: C14.2, U4.2 (REF)
- new net: C15.2, U4.3 (SS)
Other:
- note added: "3.3V step down from 4.8V"
- note added: "schottky dioda >10V reverse a co nejmin forward voltage"
- moved on the sheet: D2, R5, U3-stabilizer

Commit message: choose more values on the power circuits on the PCB
Parts:
- removed D1: D, symbol Device:D
- added D1: D_Schottky, symbol Device:D_Schottky
- added R6: 102k, symbol Device:R
- R1: value R -> 5k
- R2: value R -> 649R
- R3: value R -> 7.5k
Connections:
- net +4.8V: no longer C12.2, C13.1, C2.1, L1.2, R1.1, R5.1, U4.1 (SHDN), U4.8 (VCC)
- net GND: now also D1.2 (A)
- net at L1.1, U2.1 (OUT): now also D1.1 (K)
- net at C4.2, R1.2, R2.1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: now also R6.2
- new net +5V: C12.2, C13.1, C2.1, L1.2, R1.1, R5.1, R6.1, U4.1 (SHDN), U4.8 (VCC)
Other:
- note added: "SERVO CONTROL"
- note added: "STEP DOWN FROM 5V TO 3.3V"
- note added: "STEP DOWN FROM BATTER 12.6V TO 5V"
- note added: "schottky dioda >60V reverse a co nejmin forward voltage a proud >3A (radsi vic)"
- note removed: "3.3V step down from 4.8V"
- note removed: "4.8V step down from battery"
- moved on the sheet: C2, R1
